File: hardware/schematic-pcb/snowflake-hw-v1.0.1/snowflake-hw-v1.0.1 R5.brd (EAGLE design)
At the start: 112.6 x 138.7 mm, 180 parts, among them IC1 74AHC1G125, Q2 2N7002, Q3 IRLML6401, Q4 nc, U1 P2, U2 MP34DT05TR-A, U3 XC6220B331PR-G, U4 APX803L20-41SA, U5 RT9818C-30GV, U6 TPA6211A1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

Commit message: Add final HW files to repo
Copied files from snowflake-hw repo.
Parts:
- B1: value 220R -> 120R
- C21: value 100uF, 6.3V -> NC
- C52, C58: value 2.2uF -> 33nF
- C61: value 1000F -> 1000pF
- C69: value 100uF nc -> 100uF
- CONN1: value CONN5X2 -> CONN5X2 nc
- D2: value NC -> 1N5817W
- D3: value LXES15AAA1-133 -> LXES15AAA1-153
- D4, D5: value nc -> LXES15AAA1-153
- D6: value LRB551V-30 nc -> nc
- R25: value 10k -> 10K
- R41: value NCP18WF104F12RB -> ERTJ1VR104FM
- U$1: value SEPAKER -> NC
- U$5: value SEPAKER15X15MM -> FS-1540
Other:
- board text added: "CCSH-W10-04"
- board text added: "FS-1540"
- board text added: "TS-1185A"
- board text added: "U$1"
- board text added: "U$5"
- board text added: "nc"
- board text removed: "FS-1340"
